Commit message: thicker and random cardboard box

File: examples/cardboard_box.urdf (robot description, URDF)
Before this commit: robot cardboard_box, 5 links, 4 joints
Links:
- link back_major_flap: geometry collision box size=0.3 0.005 0.1; visual box size=0.3 0.005 0.1
- link base: geometry collision box size=0.005 0.2 0.2; collision box size=0.005 0.2 0.2
- link front_major_flap: geometry collision box size=0.3 0.005 0.1; visual box size=0.3 0.005 0.1
- link left_minor_flap: geometry collision box size=0.005 0.2 0.1; visual box size=0.005 0.2 0.1
- link right_minor_flap: geometry collision box size=0.005 0.2 0.1; visual box size=0.005 0.2 0.1
