Commit message: headless, num_envs=4, added requirements.txt

File: examples/test.urdf (robot description, URDF)
Before this commit: robot static, 30 links, 29 joints
Links:
- link center_cam_link: geometry collision box size=0.026 0.124 0.029; visual mesh filename=/home/straw/Projects/garage/sims_core/examples/meshes/camer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 scale=0.001 0.001 0.001
- link left_base_link: geometry collision mesh filename=/home/straw/Projects/garage/sims_core/examples/meshes/piper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; visual mesh filename=/home/straw/Projects/garage/sims_core/examples/meshes/piper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
- link left_cam_link: geometry collision box size=0.023 0.042 0.042; visual mesh filename=/home/straw/Projects/garage/sims_core/examples/meshes/camer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 scale=0.001 0.001 0.001
- link left_link1: geometry collision mesh filename=/home/straw/Projects/garage/sims_core/examples/meshes/piper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; visual mesh filename=/home/straw/Projects/garage/sims_core/examples/meshes/piper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
- link left_link2: geometry collision mesh filename=/home/straw/Projects/garage/sims_core/examples/meshes/piper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; visual mesh filename=/home/straw/Projects/garage/sims_core/examples/meshes/piper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
- link left_link3: geometry collision mesh filename=/home/straw/Projects/garage/sims_core/examples/meshes/piper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; visual mesh filename=/home/straw/Projects/garage/sims_core/examples/meshes/piper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
- link left_link4: geometry collision mesh filename=/home/straw/Projects/garage/sims_core/examples/meshes/piper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; visual mesh filename=/home/straw/Projects/garage/sims_core/examples/meshes/piper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
- link left_link5: geometry collision mesh filename=/home/straw/Projects/garage/sims_core/examples/meshes/piper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; visual mesh filename=/home/straw/Projects/garage/sims_core/examples/meshes/piper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
- link left_link6: geometry collision mesh filename=/home/straw/Projects/garage/sims_core/examples/meshes/piper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; visual mesh filename=/home/straw/Projects/garage/sims_core/examples/meshes/piper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
- link left_link7.1: geometry collision mesh filename=/home/straw/Projects/garage/sims_core/examples/meshes/piper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; visual mesh filename=/home/straw/Projects/garage/sims_core/examples/meshes/piper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
- link left_link7.2: geometry collision mesh filename=/home/straw/Projects/garage/sims_core/examples/meshes/piper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; visual mesh filename=/home/straw/Projects/garage/sims_core/examples/meshes/piper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
- link right_base_link: geometry collision mesh filename=/home/straw/Projects/garage/sims_core/examples/meshes/piper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; visual mesh filename=/home/straw/Projects/garage/sims_core/examples/meshes/piper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
- link right_cam_link: geometry collision box size=0.023 0.042 0.042; visual mesh filename=/home/straw/Projects/garage/sims_core/examples/meshes/camer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 scale=0.001 0.001 0.001
- link right_link1: geometry collision mesh filename=/home/straw/Projects/garage/sims_core/examples/meshes/piper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; visual mesh filename=/home/straw/Projects/garage/sims_core/examples/meshes/piper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
- link right_link2: geometry collision mesh filename=/home/straw/Projects/garage/sims_core/examples/meshes/piper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; visual mesh filename=/home/straw/Projects/garage/sims_core/examples/meshes/piper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
- link right_link3: geometry collision mesh filename=/home/straw/Projects/garage/sims_core/examples/meshes/piper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; visual mesh filename=/home/straw/Projects/garage/sims_core/examples/meshes/piper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
- link right_link4: geometry collision mesh filename=/home/straw/Projects/garage/sims_core/examples/meshes/piper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; visual mesh filename=/home/straw/Projects/garage/sims_core/examples/meshes/piper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
- link right_link5: geometry collision mesh filename=/home/straw/Projects/garage/sims_core/examples/meshes/piper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; visual mesh filename=/home/straw/Projects/garage/sims_core/examples/meshes/piper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
- link right_link6: geometry collision mesh filename=/home/straw/Projects/garage/sims_core/examples/meshes/piper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; visual mesh filename=/home/straw/Projects/garage/sims_core/examples/meshes/piper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
- link right_link7.1: geometry collision mesh filename=/home/straw/Projects/garage/sims_core/examples/meshes/piper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; visual mesh filename=/home/straw/Projects/garage/sims_core/examples/meshes/piper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
- link right_link7.2: geometry collision mesh filename=/home/straw/Projects/garage/sims_core/examples/meshes/piper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; visual mesh filename=/home/straw/Projects/garage/sims_core/examples/meshes/piper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
- link table_corner: geometry collision mesh filename=/home/straw/Projects/garage/sims_core/examples/meshes/workc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 scale=0.001 0.001 0.001; visual mesh filename=/home/straw/Projects/garage/sims_core/examples/meshes/workc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 scale=0.001 0.001 0.001
